Commit message: update terrain exps

File: amp/data/robot/h1_update/urdf/h1.urdf (robot description, URDF)
Before this commit: robot h1_description, 22 links, 21 joints
Links:
- link left_ankle_link: geometry collision box size=0.28 0.03 0.024; visual mesh filename=../meshes/left_ankle_link.STL
- link right_ankle_link: geometry collision box size=0.28 0.03 0.024; visual mesh filename=../meshes/right_ankle_link.STL

Commit message: add unitree dataset

File: amp/data/robot/h1_update/urdf/h1.urdf (robot description, URDF)
Before this commit: robot h1_description, 22 links, 21 joints
Links:
- added link left_hand_link, mass 0.014; collision mesh filename=../meshes/left_hand_link.STL; visual mesh filename=../meshes/left_hand_link.dae
- added link right_hand_link, mass 0.014; collision mesh filename=../meshes/right_hand_link.STL; visual mesh filename=../meshes/right_hand_link.dae
- link left_ankle_link: geometry collision box size=0.29 0.03 0.026; visual mesh filename=../meshes/left_ankle_link.STL
- link left_elbow_link: mass 0.669 -> 0.723; geometry collision cylinder length=0.24 radius=0.035; visual mesh filename=../meshes/left_elbow_link.STL
- link left_hip_pitch_link: geometry collision box size=0.08 0.08 0.45; collision cylinder length=0.08 radius=0.07
- link left_hip_roll_link: geometry collision cylinder length=0.01 radius=0.02; visual mesh filename=../meshes/left_hip_roll_link.STL
- link left_hip_yaw_link: geometry collision cylinder length=0.2 radius=0.07; visual mesh filename=../meshes/left_hip_yaw_link.STL
- link left_knee_link: geometry collision box size=0.06 0.05 0.37; collision cylinder length=0.1 radius=0.05
- link left_shoulder_pitch_link: geometry collision cylinder length=0.04 radius=0.03; visual mesh filename=../meshes/left_shoulder_pitch_link.STL
- link left_shoulder_roll_link: geometry collision cylinder length=0.15 radius=0.05; visual mesh filename=../meshes/left_shoulder_roll_link.STL
- link left_shoulder_yaw_link: geometry collision cylinder length=0.18 radius=0.04; visual mesh filename=../meshes/left_shoulder_yaw_link.STL
- link logo_link: geometry visual mesh filename=../meshes/logo_link.STL
- link pelvis: geometry collision box size=0.15 0.31 0.06; visual mesh filename=../meshes/pelvis.STL
- link right_ankle_link: geometry collision box size=0.29 0.03 0.026; visual mesh filename=../meshes/right_ankle_link.STL
- link right_elbow_link: mass 0.669 -> 0.723; geometry collision cylinder length=0.24 radius=0.035; visual mesh filename=../meshes/right_elbow_link.STL
- link right_hip_pitch_link: geometry collision box size=0.08 0.08 0.45; collision cylinder length=0.08 radius=0.07
- link right_hip_roll_link: geometry collision cylinder length=0.01 radius=0.02; visual mesh filename=../meshes/right_hip_roll_link.STL
- link right_hip_yaw_link: geometry collision cylinder length=0.2 radius=0.07; visual mesh filename=../meshes/right_hip_yaw_link.STL
- link right_knee_link: geometry collision box size=0.06 0.05 0.37; collision cylinder length=0.1 radius=0.05
- link right_shoulder_pitch_link: geometry collision cylinder length=0.04 radius=0.03; visual mesh filename=../meshes/right_shoulder_pitch_link.STL
- link right_shoulder_roll_link: geometry collision cylinder length=0.15 radius=0.05; visual mesh filename=../meshes/right_shoulder_roll_link.STL
- link right_shoulder_yaw_link: geometry collision cylinder length=0.18 radius=0.04; visual mesh filename=../meshes/right_shoulder_yaw_link.STL
- link torso_link: geometry collision box size=0.12 0.3 0.14; collision box size=0.17 0.15 0.21
Joints:
- added joint left_hand_joint: type fixed, parent left_elbow_link, child left_hand_link, origin xyz=0.2605 0 -0.0185 rpy=0 0 0, axis 1 0 0, limit lower=-3.0543261909900767596164588448551 upper=3.0543261909900767596164588448551 effort=6 velocity=12
- added joint right_hand_joint: type fixed, parent right_elbow_link, child right_hand_link, origin xyz=0.2605 0 -0.0185 rpy=0 0 0, axis 1 0 0, limit lower=-3.0543261909900767596164588448551 upper=3.0543261909900767596164588448551 effort=6 velocity=12
- joint left_hip_pitch_joint: limit lower=-1.57 upper=1.57 effort=200 velocity=23 -> lower=-3.14 upper=2.53 effort=200 velocity=23
- joint right_hip_pitch_joint: limit lower=-1.57 upper=1.57 effort=200 velocity=23 -> lower=-3.14 upper=2.53 effort=200 velocity=23

Commit message: add update data formulation

File: amp/data/robot/h1_update/urdf/h1.urdf (robot description, URDF)
Before this commit: robot h1_description, 24 links, 23 joints
Links:
- link left_hip_pitch_link: geometry collision box size=0.08 0.08 0.45; collision cylinder length=0.08 radius=0.05
- link left_hip_roll_link: geometry visual mesh filename=../meshes/left_hip_roll_link.STL
- link left_hip_yaw_link: geometry visual mesh filename=../meshes/left_hip_yaw_link.STL
- link pelvis: geometry collision mesh filename=../meshes/pelvis.STL; visual mesh filename=../meshes/pelvis.STL
- link right_hip_pitch_link: geometry collision box size=0.08 0.08 0.45; collision cylinder length=0.08 radius=0.05
- link right_hip_roll_link: geometry visual mesh filename=../meshes/right_hip_roll_link.STL
- link right_hip_yaw_link: geometry visual mesh filename=../meshes/right_hip_yaw_link.STL
- link torso_link: geometry collision box size=0.12 0.3 0.1; collision box size=0.17 0.15 0.21

Commit message: add update data formulation

File: amp/data/robot/h1_update/urdf/h1.urdf (robot description, URDF)
Before this commit: robot h1_description, 24 links, 23 joints
Links:
- link left_ankle_link: geometry collision mesh filename=../meshes/left_ankle_link.STL; visual mesh filename=../meshes/left_ankle_link.STL
- link right_ankle_link: geometry collision mesh filename=../meshes/right_ankle_link.STL; visual mesh filename=../meshes/right_ankle_link.STL

Commit message: add update data formulation

File: amp/data/robot/h1_update/urdf/h1.urdf (robot description, URDF)
Before this commit: robot h1_description, 24 links, 23 joints
Links:
- link left_ankle_link: geometry collision box size=0.29 0.03 0.026; visual mesh filename=../meshes/left_ankle_link.STL
- link right_ankle_link: geometry collision box size=0.29 0.03 0.026; visual mesh filename=../meshes/right_ankle_link.STL
